File: Robot.brd (EAGLE design)
At the start: 50.8 x 50.8 mm, 22 parts, among them U1 LSM9DS0, U2 TLV1117-33CDCY

Commit message: fixed routing problem
Routing:
- net VDD: track 76.2 -> 78.8 mm
Changed lines of the file:
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@@
 <wire x1="18.2" y1="18.63" x2="19.05" y2="17.78" width="0.1524" layer="1"/>
 <via x="19.05" y="17.78" extent="1-16" drill="0.3302"/>
-<wire x1="19.05" y1="17.78" x2="19.05" y2="16.51" width="0.1524" layer="16"/>
-<wire x1="19.05" y1="16.51" x2="12.7" y2="10.16" width="0.1524" layer="16"/>
-<via x="12.7" y="10.16" extent="1-16" drill="0.3302"/>
-<wire x1="12.7" y1="10.16" x2="12.7" y2="6.975" width="0.1524" layer="1"/>
+<via x="12.7" y="8.128" extent="1-16" drill="0.3302"/>
+<wire x1="12.7" y1="8.128" x2="12.7" y2="6.975" width="0.1524" layer="1"/>
 <wire x1="12.7" y1="6.975" x2="12.72" y2="6.955" width="0.1524" layer="1"/>
+<wire x1="19.05" y1="17.78" x2="19.05" y2="14.478" width="0.1524" layer="16"/>
+<wire x1="19.05" y1="14.478" x2="12.7" y2="8.128" width="0.1524" layer="16"/>
 </signal>
 <signal name="SCL">
@@
 <wire x1="17.78" y1="20.74" x2="16.76" y2="19.72" width="0.1524" layer="1"/>
 <wire x1="16.76" y1="19.72" x2="15.87" y2="19.72" width="0.1524" layer="1"/>
-<wire x1="14.22" y1="6.955" x2="14.22" y2="9.14" width="0.1524" layer="1"/>
-<wire x1="14.22" y1="9.14" x2="15.24" y2="10.16" width="0.1524" layer="1"/>
-<via x="15.24" y="10.16" extent="1-16" drill="0.3302"/>
-<wire x1="15.24" y1="10.16" x2="20.32" y2="15.24" width="0.1524" layer="16"/>
-<wire x1="20.32" y1="15.24" x2="20.32" y2="19.05" width="0.1524" layer="16"/>
+<via x="14.224" y="8.128" extent="1-16" drill="0.3302"/>
+<wire x1="20.32" y1="14.224" x2="20.32" y2="19.05" width="0.1524" layer="16"/>
 <via x="20.32" y="19.05" extent="1-16" drill="0.3302"/>
 <wire x1="20.32" y1="19.05" x2="19.47" y2="19.05" width="0.1524" layer="1"/>
 <wire x1="19.47" y1="19.05" x2="17.78" y2="20.74" width="0.1524" layer="1"/>
+<wire x1="14.22" y1="6.955" x2="14.22" y2="8.124" width="0.1524" layer="1"/>
+<wire x1="14.22" y1="8.124" x2="14.224" y2="8.128" width="0.1524" layer="1"/>
+<wire x1="20.32" y1="14.224" x2="14.224" y2="8.128" width="0.1524" layer="16"/>
 </signal>
 <signal name="GND" airwireshidden="yes">
@@
 <wire x1="17.78" y1="3.39" x2="17.36" y2="3.81" width="0.1524" layer="1"/>
 <wire x1="17.36" y1="3.81" x2="16.51" y2="3.81" width="0.1524" layer="1"/>
-<wire x1="10.16" y1="8.47" x2="13.705" y2="8.47" width="0.1524" layer="1"/>
-<wire x1="13.705" y1="8.47" x2="15.22" y2="6.955" width="0.1524" layer="1"/>
 <wire x1="41.28" y1="31.75" x2="39.37" y2="31.75" width="0.1524" layer="1"/>
 <wire x1="39.37" y1="31.75" x2="38.1" y2="30.48" width="0.1524" layer="1"/>
@@
 <wire x1="17.78" y1="22.44" x2="24.55" y2="22.44" width="0.1524" layer="1"/>
 <wire x1="24.55" y1="22.44" x2="26.3398" y2="20.6502" width="0.1524" layer="1"/>
+<wire x1="10.16" y1="8.47" x2="11.01" y2="8.47" width="0.1524" layer="1"/>
+<wire x1="11.01" y1="8.47" x2="12.7" y2="10.16" width="0.1524" layer="1"/>
+<wire x1="12.7" y1="10.16" x2="13.97" y2="10.16" width="0.1524" layer="1"/>
+<wire x1="13.97" y1="10.16" x2="15.24" y2="8.89" width="0.1524" layer="1"/>
+<wire x1="15.24" y1="8.89" x2="15.24" y2="6.975" width="0.1524" layer="1"/>
+<wire x1="15.24" y1="6.975" x2="15.22" y2="6.955" width="0.1524" layer="1"/>
 </signal>
 <signal name="N$4">

Commit message: ALmost done with layout
Parts:
- added C11, C12, C14: 0.1uF, SparkFun-Capacitors:0603-CAP
- added C13: 47nF, SparkFun-Capacitors:0603-CAP
- added C15: 1nF, SparkFun-Capacitors:0603-CAP
- added C16: 1.0uF, SparkFun-Capacitors:0603-CAP
- added C17: 100pF, SparkFun-Capacitors:0603-CAP
- added D2, D3: 1N4004, diode:DO41-10
- added JP1, JP4: (no value), SparkFun-Connectors:1X04
- added JP2, JP3, JP6: M02PTH, SparkFun-Connectors:1X02
- added JP5: (no value), SparkFun-Connectors:1X05
- added R10, R8, R9: 1K, SparkFun-Resistors:0603-RES
- added R11, R5: 100k, SparkFun-Resistors:0603-RES
- added R4: 10K, SparkFun-Resistors:0603-RES
- added T1, T2: (no value), zetex:SOT-23
- added U$4: BALUN-2450BM, NordicSemi:2450BM14A0002
- added U$6: OPA344, SparkFun-AnalogIC:SOT23-5
- R1, R2: value 100k -> 4.7K
- moved U$5 36.2 mm to (48.8, 27.8), turned to 90 degrees
- moved C5 32.3 mm to (47.8, 31.0), turned to 0 degrees
- moved C6 27.3 mm to (42.4, 26.5), turned to 180 degrees
- moved R3 18.6 mm to (20.1, 40.0), turned to 0 degrees
- moved R1 17.7 mm to (21.6, 17.8), turned to 180 degrees
- moved J1 16.3 mm to (46.6, 7.87)
- moved C7 16.3 mm to (44.6, 15.5)
- moved C8 16.3 mm to (31.9, 1.52)
- moved D1 16.3 mm to (38.2, 6.60)
- moved U2 16.3 mm to (31.9, 6.60)
- moved U$2 10.2 mm to (1.65, 14.0), turned to 270 degrees
- moved R2 4.58 mm to (21.6, 20.3), turned to 180 degrees
Connections:
- removed net MOTOR3: U$1.8
- removed net MOTOR4: U$1.9
- new net N$10: C14.1, U$1.39
- new net N$11: U$1.32, U$4.4
- new net N$12: U$1.31, U$4.3
- new net N$13: U$1.30, U$4.5
- new net N$14: U$2.FP, U$4.1
- new net N$15: D2.A, JP2.2, T1.1
- new net N$16: D3.A, JP3.2, T2.1
- new net N$19: C6.2, R8.1
- new net N$20: C16.1, R10.2, R9.1, U$6.3
- new net N$22: C17.1, R11.1, R8.2, U$6.4
- new net N$7: C13.1, U$1.29
- new net RX: JP6.1, U$1.18
- new net SDWIO: JP1.3, U$1.23
- new net SWDCLK: JP1.2, U$1.24
- new net TX: JP6.2, U$1.17
- net GND: now also C11.2, C12.2, C13.2, C14.2, C15.2, C16.2, JP1.1, JP4.1, JP4.2, JP4.3, JP4.4, R10.1, R3.2, R5.2, T1.2, T2.2, U$1.13, U$1.33, U$1.34, U$1.GND, U$4.2, U$6.2, U1.22, U1.23
- net MIC: now also C17.2, JP5.1, R11.2, U$6.1; no longer C6.2
- net MOTOR1: now also JP5.3, R3.1, T1.3
- net MOTOR2: now also JP5.2, R5.1, T2.3
- net N$4: now also R4.1; no longer R1.1
- net SCL: now also JP5.4, R2.2; no longer R3.2
- net SDA: now also JP5.5, R1.2; no longer R2.2
- net VDD: now also C11.1, C12.1, C15.1, D2.C, D3.C, JP1.4, JP2.1, JP3.1, R1.1, R4.2, R9.2, U$1.1, U$1.12, U$1.35, U$1.36, U$6.5; no longer R1.2, R3.1
Routing:
- net VDD: track 78.8 -> 163.3 mm, vias 0 -> 6
- net MIC: track 12.9 -> 45.7 mm
- net RX: track 0.00 -> 11.1 mm, vias 0 -> 1
- net N$15: track 0.00 -> 11.0 mm
- net N$16: track 0.00 -> 10.8 mm
- net N$22: track 0.00 -> 8.48 mm
- net N$20: track 0.00 -> 8.16 mm
- net TX: track 0.00 -> 7.64 mm, vias 0 -> 1
- net N$14: track 0.00 -> 7.19 mm
- net SDWIO: track 0.00 -> 6.89 mm
- net SWDCLK: track 0.00 -> 6.00 mm
- net N$12: track 0.00 -> 5.80 mm, vias 0 -> 2
- net GND: track 0.00 -> 5.73 mm, vias 2 -> 7
- net N$10: track 0.00 -> 4.91 mm, vias 0 -> 2
- net N$11: track 0.00 -> 4.26 mm
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
Commit message: Finished layout
Parts:
- moved U$2 11.0 mm to (1.65, 2.92)
- moved JP4 5.00 mm to (2.03, 32.8), turned to 90 degrees
Routing:
- net MOTOR1: track 2.02 -> 48.5 mm, vias 0 -> 1
- net MOTOR2: track 1.96 -> 37.7 mm
- net SCL: track 20.8 -> 37.7 mm
- net SDA: track 19.7 -> 34.4 mm
- net N$14: track 7.19 -> 18.2 mm
- net MIC: track 45.7 -> 56.5 mm
- net GND: vias 7 -> 34
Other:
- board text added: "GND"

Commit message: Working on silk screen
Parts:
- renumbered U$2 to ANT1
Other:
- board text added: "ANT1"
- board text added: "C1"
- board text added: "C2"
- board text added: "C3"
- board text added: "C4"
- board text added: "C8"
- board text added: "MIC"
- board text added: "MOTOR1"
- board text added: "MOTOR2"
- board text added: "R4"
- board text added: "RX"
- board text added: "SCL"
- board text added: "SDA"
- board text added: "SWDCLK"
- board text added: "SWDIO"
- board text added: "TX"
- board text added: "U1"
- board text added: "U2"
- board text added: "VDD"
Changed lines of the file:
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@@
 <?xml version="1.0" encoding="utf-8"?>
 <!DOCTYPE eagle SYSTEM "eagle.dtd">
-<eagle version="7.2.0">
+<eagle version="6.5.0">
 <drawing>
 <settings>
@@
 <setting verticaltext="up"/>
 </settings>
-<grid distance="0.05" unitdist="inch" unit="inch" style="lines" multiple="1" display="yes" altdistance="0.005" altunitdist="inch" altunit="inch"/>
+<grid distance="0.005" unitdist="inch" unit="inch" style="lines" multiple="1" display="yes" altdistance="0.005" altunitdist="inch" altunit="inch"/>
 <layers>
 <layer number="1" name="Top" color="4" fill="1" visible="yes" active="yes"/>
@@
 <layer number="23" name="tOrigins" color="15" fill="1" visible="yes" active="yes"/>
 <layer number="24" name="bOrigins" color="15" fill="1" visible="yes" active="yes"/>
-<layer number="25" name="tNames" color="7" fill="1" visible="yes" active="yes"/>
+<layer number="25" name="tNames" color="7" fill="1" visible="no" active="yes"/>
 <layer number="26" name="bNames" color="7" fill="1" visible="yes" active="yes"/>
-<layer number="27" name="tValues" color="7" fill="1" visible="yes" active="yes"/>
+<layer number="27" name="tValues" color="7" fill="1" visible="no" active="yes"/>
 <layer number="28" name="bValues" color="7" fill="1" visible="yes" active="yes"/>
 <layer number="29" name="tStop" color="7" fill="3" visible="no" active="yes"/>
@@
 <layer number="116" name="Patch_BOT" color="9" fill="4" visible="yes" active="yes"/>
 <layer number="121" name="_tsilk" color="7" fill="1" visible="yes" active="yes"/>
-<layer number="122" name="_bsilk" color="7" fill="1" visible="yes" active="yes"/>
+<layer number="122" name="_bsilk" color="7" fill="1" visible="no" active="yes"/>
 <layer number="123" name="tTestmark" color="7" fill="1" visible="yes" active="yes"/>
 <layer number="124" name="bTestmark" color="7" fill="1" visible="yes" active="yes"/>
@@
 <wire x1="50.8" y1="50.8" x2="50.8" y2="0" width="0.4064" layer="20"/>
 <wire x1="50.8" y1="0" x2="0" y2="0" width="0.4064" layer="20"/>
-<text x="3.556" y="39.624" size="1.524" layer="112">GND</text>
-<text x="3.556" y="36.957" size="1.524" layer="112">GND</text>
-<text x="3.556" y="34.544" size="1.524" layer="112">GND</text>
-<text x="3.556" y="32.004" size="1.524" layer="112">GND</text>
+<text x="29.21" y="24.13" size="0.762" layer="121">MIC</text>
+<text x="26.67" y="21.59" size="0.762" layer="121">MOTOR2</text>
+<text x="26.67" y="19.05" size="0.762" layer="121">MOTOR1</text>
+<text x="29.21" y="16.51" size="0.762" layer="121">SCL</text>
+<text x="29.21" y="13.97" size="0.762" layer="121">SDA</text>
+<text x="3.81" y="39.37" size="0.762" layer="121">GND</text>
+<text x="3.81" y="36.83" size="0.762" layer="121">GND</text>
+<text x="3.81" y="34.29" size="0.762" layer="121">GND</text>
+<text x="3.81" y="31.75" size="0.762" layer="121">GND</text>
+<text x="9.017" y="30.861" size="0.762" layer="121" rot="R90">GND</text>
+<text x="11.557" y="30.861" size="0.762" layer="121" rot="R90">SWDCLK</text>
+<text x="14.097" y="30.861" size="0.762" layer="121" rot="R90">SWDIO</text>
+<text x="16.637" y="30.861" size="0.762" layer="121" rot="R90">VDD</text>
+<text x="20.701" y="28.956" size="0.762" layer="121">RX</text>
+<text x="20.701" y="26.289" size="0.762" layer="121">TX</text>
+<text x="2.667" y="4.191" size="0.762" layer="121" rot="R270">ANT1</text>
+<text x="9.017" y="6.858" size="0.762" layer="121" rot="R90">C3</text>
+<text x="9.017" y="3.048" size="0.762" layer="121" rot="R90">C2</text>
+<text x="10.922" y="2.032" size="0.762" layer="121">C1</text>
+<text x="14.605" y="1.905" size="0.762" layer="121">R4</text>
+<text x="18.923" y="3.048" size="0.762" layer="121" rot="R270">C4</text>
+<text x="13.335" y="7.493" size="0.762" layer="121">U1</text>
+<text x="31.115" y="10.287" size="0.762" layer="121">U2</text>
+<text x="31.242" y="2.286" size="0.762" layer="121">C8</text>
 </plain>
 <attributes>
@@
 </class>
 </classes>
-<designrules name="LaenPCBOrder">
+<designrules name="OshPark">
 <description language="de">&lt;b&gt;EAGLE Design Rules&lt;/b&gt;
 &lt;p&gt;
@@
 <pass name="Default">
 <param name="RoutingGrid" value="50mil"/>
-<param name="AutoGrid" value="1"/>
-<param name="Efforts" value="0"/>
-<param name="TopRouterVariant" value="1"/>
 <param name="tpViaShape" value="round"/>
-<param name="PrefDir.1" value="a"/>
+<param name="PrefDir.1" value="|"/>
 <param name="PrefDir.2" value="0"/>
 <param name="PrefDir.3" value="0"/>
@@
 <param name="PrefDir.14" value="0"/>
 <param name="PrefDir.15" value="0"/>
-<param name="PrefDir.16" value="a"/>
+<param name="PrefDir.16" value="-"/>
 <param name="cfVia" value="8"/>
 <param name="cfNonPref" value="5"/>
@@
 <element name="FRAME1" library="SparkFun-Aesthetics" package="CREATIVE_COMMONS" value="FRAME-LETTER" x="-77.47" y="25.4"/>
 <element name="U$1" library="NordicSemi" package="QFN48" value="NRF51822" x="12.7" y="20.32" rot="R180"/>
-<element name="U$2" library="NordicSemi" package="2450AT18B100" value="ANTENA-2450AT" x="1.651" y="2.921" rot="R270"/>
+<element name="ANT1" library="NordicSemi" package="2450AT18B100" value="ANTENA-2450AT" x="1.651" y="2.921" rot="R270"/>
 <element name="U$3" library="NordicSemi" package="2.5X2MM" value="CRYSTAL2.5X2" x="10.16" y="13.97"/>
 <element name="U$5" library="SparkFun-Sensors" package="ADMP401" value="ADMP401" x="48.768" y="27.813" rot="R90"/>
@@
 <signal name="N$14">
 <contactref element="U$4" pad="1"/>
-<contactref element="U$2" pad="FP"/>
+<contactref element="ANT1" pad="FP"/>
 <wire x1="4.505" y1="20.82" x2="3.04" y2="20.82" width="0.1524" layer="1"/>
 <wire x1="3.04" y1="20.82" x2="1.651" y2="19.431" width="0.1524" layer="1" curve="90"/>
